Commit message: Fixed rviz visualization; Fixed bug in kinect xacro

File: lubobot/urdf/kinect.urdf.xacro (robot description, xacro)
@@ -21,5 +21,5 @@
         <origin xyz="-0.05 -0.17 -0.02" rpy="${3.1415/2.0} 0 ${3.1415/2.0}"/>
         <geometry>
-          <mesh filename="package://lubobot/kinect/meshes/68-04546_Kinect_Sensor--coarse_simple.STL" scale="0.001 0.001 0.001" />
+          <mesh filename="package://lubobot/meshes/kinect/68-04546_Kinect_Sensor--coarse_simple.STL" scale="0.001 0.001 0.001" />
         </geometry>
       </collision>

File: lubobot/urdf/lubobot.urdf.xacro (robot description, xacro)
@@ -6,11 +6,6 @@
 		<mesh filename="package://lubobot/meshes/create_2.dae" />
 	</xacro:create_base>
-	<!-- shoulder kinect -->
-	<!-- ORIGINAL DATA FROM HALCON CALIBRATION:
-             from: base_link to: shoulder_kinect_link
-             translation: -0.135394 -0.00764754 1.54755 (xyz)
-             quaternion: 0.0177781 0.202257 -0.0472198 0.978032 (xyzw) -->
 	<kinect name="shoulder_kinect" parent="base_link">
-		<origin xyz="-0.135394 -0.00764754 1.54755" rpy="0.01708077682636155 0.4085798647123734 -0.09294704527264909"/>
+		<origin xyz="0 0 0.3" rpy="0 0 0"/>
 	</kinect>
 </robot>
