Commit message: WIP: body urdf

File: lubobot/urdf/body.urdf.xacro (robot description, xacro)
@@ -2,26 +2,55 @@
 <robot name="body"
   xmlns:xacro="http://ros.org/wiki/xacro">
-  <xacro:macro name="body" params="parent *origin">
-    <joint name="${name}_joint" type="fixed">
-      <xacro:insert_block name="origin"/>
+  <!-- Heavily based on: https://github.com/turtlebot/turtlebot/blob/5a97fdd2661354a866ee41238e2197244c220840/turtlebot_description/urdf/stacks/hexagons.urdf.xacro -->
+  <xacro:macro name="stack_bottom_pole" params="parent number x_loc y_loc z_loc">
+    <joint name="pole_bottom_${number}_joint" type="fixed">
+      <origin xyz="${x_loc} ${y_loc} ${z_loc}" rpy="0 0 0"/>
       <parent link="${parent}"/>
-      <child link="${name}_link" />
+      <child link="pole_bottom_${number}_link"/>
     </joint>
-    <link name="${name}_link">
+    <link name="pole_bottom_${number}_link">
       <visual>
-        <origin xyz="-0.05 -0.17 -0.02" rpy="${3.1415/2.0} 0 ${3.1415/2.0}"/>
+        <origin xyz="0 0 0" rpy="0 0 0"/>
         <geometry>
-          <mesh filename="package://lubobot/meshes/kinect/68-04546_Kinect_Sensor--coarse.STL" scale="0.001 0.001 0.001" />
+          <mesh filename="package://turtlebot_description/meshes/stacks/hexagons/pole_bottom.dae"/>
         </geometry>
-        <material name="gray">
-          <color rgba="0.5 0.5 0.5 1"/>
-        </material>
       </visual>
       <collision>
-        <origin xyz="-0.05 -0.17 -0.02" rpy="${3.1415/2.0} 0 ${3.1415/2.0}"/>
+        <origin xyz="0 0 0" rpy="0 0 0"/>
         <geometry>
-          <mesh filename="package://lubobot/meshes/kinect/68-04546_Kinect_Sensor--coarse_simple.STL" scale="0.001 0.001 0.001" />
+          <cylinder length="0.0492" radius="0.006"/>
         </geometry>
       </collision>
+      <inertial>
+        <mass value="0.008"/>
+        <origin xyz="0 0 0" rpy="0 0 0"/>
+        <inertia ixx="0.000001686" ixy="0.0" ixz="0.0" iyy="0.000001686" iyz="0.0" izz="0.000000144"/>
+      </inertial>
+    </link>
+  </xacro:macro>
+  <xacro:macro name="stack_top_pole" params="parent number x_loc y_loc z_loc">
+    <joint name="pole_top_${number}_joint" type="fixed">
+      <origin xyz="${x_loc} ${y_loc} ${z_loc}" rpy="0 0 0"/>
+      <parent link="${parent}"/>
+      <child link="pole_top_${number}_link"/>
+    </joint>
+    <link name="pole_top_${number}_link">
+      <visual>
+        <origin xyz=" 0 0 0" rpy="0 0 0"/>
+        <geometry>
+          <mesh filename="package://turtlebot_description/meshes/stacks/hexagons/pole_top.dae"/>
+        </geometry>
+      </visual>
+      <collision>
+        <origin xyz="0 0 0" rpy="0 0 0"/>
+        <geometry>
+          <cylinder length="0.2032" radius="0.006"/>
+        </geometry>
+      </collision>
+      <inertial>
+        <mass value="0.060"/>
+        <origin xyz="0 0 0"/>
+        <inertia ixx="0.000206991" ixy="0.0" ixz="0.0" iyy="0.000206991" iyz="0.0" izz="0.000001080"/>
+      </inertial>
     </link>
   </xacro:macro>

Commit message: Robot model starts to make sense

File: lubobot/urdf/body.urdf.xacro (robot description, xacro)
@@ -13,5 +13,5 @@
         <origin xyz="0 0 0" rpy="0 0 0"/>
         <geometry>
-          <mesh filename="package://turtlebot_description/meshes/stacks/hexagons/pole_bottom.dae"/>
+          <mesh filename="package://lubobot/meshes/pole_100mm.stl" scale="0.001 0.001 0.001"/>
         </geometry>
       </visual>
@@ -19,5 +19,5 @@
         <origin xyz="0 0 0" rpy="0 0 0"/>
         <geometry>
-          <cylinder length="0.0492" radius="0.006"/>
+          <mesh filename="package://lubobot/meshes/pole_100mm.stl" scale="0.001 0.001 0.001"/>
         </geometry>
       </collision>
@@ -39,11 +39,11 @@
         <origin xyz=" 0 0 0" rpy="0 0 0"/>
         <geometry>
-          <mesh filename="package://turtlebot_description/meshes/stacks/hexagons/pole_top.dae"/>
+          <mesh filename="package://lubobot/meshes/pole_100mm.stl" scale="0.001 0.001 0.001"/>
         </geometry>
       </visual>
       <collision>
-        <origin xyz="0 0 0" rpy="0 0 0"/>
+        <origin xyz=" 0 0 0" rpy="0 0 0"/>
         <geometry>
-          <cylinder length="0.2032" radius="0.006"/>
+          <mesh filename="package://lubobot/meshes/pole_100mm.stl" scale="0.001 0.001 0.001"/>
         </geometry>
       </collision>
@@ -55,3 +55,66 @@
     </link>
   </xacro:macro>
+  <!--
+    Stack macro - all the components relative transforms are made with respect
+    to the parent link (usually base_link). They could be made relative to each
+    other, but there is no necessary reason to do so.
+  -->
+  <xacro:macro name="body" params="parent">
+    <xacro:stack_bottom_pole parent="${parent}" number="0" x_loc= "0.120" y_loc= "0.082" z_loc="0.1028"/>
+    <xacro:stack_bottom_pole parent="${parent}" number="1" x_loc= "0.055" y_loc= "0.120" z_loc="0.1028"/>
+    <xacro:stack_bottom_pole parent="${parent}" number="2" x_loc="-0.055" y_loc= "0.120" z_loc="0.1028"/>
+    <xacro:stack_bottom_pole parent="${parent}" number="3" x_loc= "0.120" y_loc="-0.082" z_loc="0.1028"/>
+    <joint name="plate_bottom_joint" type="fixed">
+      <origin xyz="0.02364 0.0 0.1306" rpy="0 0 0"/>
+      <parent link="${parent}"/>
+      <child link="plate_bottom_link"/>
+    </joint>
+    <link name="plate_bottom_link">
+      <visual>
+        <origin xyz="0 0 0" rpy="0 0 0"/>
+        <geometry>
+          <mesh filename="package://lubobot/meshes/bottom_plate_290mm.stl" scale="0.001 0.001 0.001"/>
+        </geometry>
+      </visual>
+      <collision>
+        <origin xyz="0 0 0" rpy="0 0 0"/>
+        <geometry>
+          <mesh filename="package://lubobot/meshes/bottom_plate_290mm.stl" scale="0.001 0.001 0.001"/>
+        </geometry>
+      </collision>
+      <inertial>
+        <mass value="0.520" />
+        <origin xyz="0 0 0" />
+        <inertia ixx="0.003328" ixy="0.0" ixz="0.0" iyy="0.003328" iyz="0.0" izz="0.006656" />
+      </inertial>
+    </link>
+    <xacro:stack_top_pole parent="${parent}" number="0" x_loc= "0.0381" y_loc= "0.1505" z_loc="0.2920"/>
+    <xacro:stack_top_pole parent="${parent}" number="1" x_loc= "0.0381" y_loc="-0.1505" z_loc="0.2920"/>
+    <xacro:stack_top_pole parent="${parent}" number="2" x_loc="-0.0381" y_loc= "0.1505" z_loc="0.2920"/>
+    <xacro:stack_top_pole parent="${parent}" number="3" x_loc="-0.0381" y_loc="-0.1505" z_loc="0.2920"/>
+    <joint name="plate_top_joint" type="fixed">
+      <origin xyz="-0.01364 0.0  0.3966" rpy="0 0 0"/>
+      <parent link="${parent}"/>
+      <child link="plate_top_link"/>
+    </joint>
+    <link name="plate_top_link">
+      <visual>
+        <origin xyz="0 0 0" rpy="0 0 0"/>
+        <geometry>
+          <mesh filename="package://lubobot/meshes/top_plate_290mm.stl" scale="0.001 0.001 0.001"/>
+        </geometry>
+      </visual>
+      <collision>
+        <origin xyz="0 0 0" rpy="0 0 0"/>
+        <geometry>
+          <mesh filename="package://lubobot/meshes/top_plate_290mm.stl" scale="0.001 0.001 0.001"/>
+        </geometry>
+      </collision>
+      <inertial>
+        <mass value="0.520"/>
+        <origin xyz="0 0 0"/>
+        <inertia ixx="0.003328" ixy="0.0" ixz="0.0" iyy="0.003328" iyz="0.0" izz="0.006656" />
+      </inertial>
+    </link>
+  </xacro:macro>
 </robot>

File: lubobot/urdf/lubobot.urdf.xacro (robot description, xacro)
@@ -8,11 +8,8 @@
 		<mesh filename="package://lubobot/meshes/create_2.dae" />
 	</xacro:create_base>
-	<xacro:body parent="base_link">
-		<origin xyz="0 0 0" rpy="0 0 0"/>
-	</xacro:body>
+	<xacro:body parent="base_link"/>
 	<xacro:kinect name="camera" parent="base_link">
 		<origin xyz="0 0 0.3" rpy="0 0 0"/>
 	</xacro:kinect>
-	<!-- <xacro:imu_sensor xyz="-0.1 0 0.07" rpy="0 0 0" parent="base_link" /> -->
 	<xacro:imu_sensor xyz="0 0 0" rpy="0 0 -1.57075" parent="base_link" />
 </robot>

Commit message: Basic URDF finished

File: lubobot/urdf/body.urdf.xacro (robot description, xacro)
@@ -13,5 +13,5 @@
         <origin xyz="0 0 0" rpy="0 0 0"/>
         <geometry>
-          <mesh filename="package://lubobot/meshes/pole_100mm.stl" scale="0.001 0.001 0.001"/>
+          <mesh filename="package://lubobot/meshes/pole_80mm.stl" scale="0.001 0.001 0.001"/>
         </geometry>
       </visual>
@@ -19,5 +19,5 @@
         <origin xyz="0 0 0" rpy="0 0 0"/>
         <geometry>
-          <mesh filename="package://lubobot/meshes/pole_100mm.stl" scale="0.001 0.001 0.001"/>
+          <mesh filename="package://lubobot/meshes/pole_80mm.stl" scale="0.001 0.001 0.001"/>
         </geometry>
       </collision>
@@ -61,10 +61,10 @@
   -->
   <xacro:macro name="body" params="parent">
-    <xacro:stack_bottom_pole parent="${parent}" number="0" x_loc= "0.120" y_loc= "0.082" z_loc="0.1028"/>
-    <xacro:stack_bottom_pole parent="${parent}" number="1" x_loc= "0.055" y_loc= "0.120" z_loc="0.1028"/>
-    <xacro:stack_bottom_pole parent="${parent}" number="2" x_loc="-0.055" y_loc= "0.120" z_loc="0.1028"/>
-    <xacro:stack_bottom_pole parent="${parent}" number="3" x_loc= "0.120" y_loc="-0.082" z_loc="0.1028"/>
+    <xacro:stack_bottom_pole parent="${parent}" number="0" x_loc= "0.08" y_loc= "0.08" z_loc="0.112"/>
+    <xacro:stack_bottom_pole parent="${parent}" number="1" x_loc= "0.08" y_loc= "-0.08" z_loc="0.112"/>
+    <xacro:stack_bottom_pole parent="${parent}" number="2" x_loc= "-0.08" y_loc= "0.08" z_loc="0.112"/>
+    <xacro:stack_bottom_pole parent="${parent}" number="3" x_loc= "-0.08" y_loc= "-0.08" z_loc="0.112"/>
     <joint name="plate_bottom_joint" type="fixed">
-      <origin xyz="0.02364 0.0 0.1306" rpy="0 0 0"/>
+      <origin xyz="0 0 0.156" rpy="0 0 0"/>
       <parent link="${parent}"/>
       <child link="plate_bottom_link"/>
@@ -89,10 +89,10 @@
       </inertial>
     </link>
-    <xacro:stack_top_pole parent="${parent}" number="0" x_loc= "0.0381" y_loc= "0.1505" z_loc="0.2920"/>
-    <xacro:stack_top_pole parent="${parent}" number="1" x_loc= "0.0381" y_loc="-0.1505" z_loc="0.2920"/>
-    <xacro:stack_top_pole parent="${parent}" number="2" x_loc="-0.0381" y_loc= "0.1505" z_loc="0.2920"/>
-    <xacro:stack_top_pole parent="${parent}" number="3" x_loc="-0.0381" y_loc="-0.1505" z_loc="0.2920"/>
+    <xacro:stack_top_pole parent="${parent}" number="0" x_loc= "0.07" y_loc= "0.10" z_loc="0.210"/>
+    <xacro:stack_top_pole parent="${parent}" number="1" x_loc= "0.07" y_loc= "-0.10" z_loc="0.210"/>
+    <xacro:stack_top_pole parent="${parent}" number="2" x_loc= "-0.07" y_loc= "0.10" z_loc="0.210"/>
+    <xacro:stack_top_pole parent="${parent}" number="3" x_loc= "-0.07" y_loc= "-0.10" z_loc="0.210"/>
     <joint name="plate_top_joint" type="fixed">
-      <origin xyz="-0.01364 0.0  0.3966" rpy="0 0 0"/>
+      <origin xyz="0 0 0.264" rpy="0 0 0"/>
       <parent link="${parent}"/>
       <child link="plate_top_link"/>

File: lubobot/urdf/lubobot.urdf.xacro (robot description, xacro)
@@ -10,6 +10,6 @@
 	<xacro:body parent="base_link"/>
 	<xacro:kinect name="camera" parent="base_link">
-		<origin xyz="0 0 0.3" rpy="0 0 0"/>
+		<origin xyz="0.050 0.033 0.210" rpy="0 0 0"/>
 	</xacro:kinect>
-	<xacro:imu_sensor xyz="0 0 0" rpy="0 0 -1.57075" parent="base_link" />
+	<xacro:imu_sensor xyz="-0.1 0 0.075" rpy="0 0 -1.57075" parent="base_link" />
 </robot>

Commit message: Simplified things to reuse as much as possible from create_autonomy

File: lubobot/urdf/body.urdf.xacro (robot description, xacro)
@@ -29,5 +29,5 @@
     </link>
   </xacro:macro>
-  <xacro:macro name="stack_top_pole" params="parent number x_loc y_loc z_loc">
+  <!-- <xacro:macro name="stack_top_pole" params="parent number x_loc y_loc z_loc">
     <joint name="pole_top_${number}_joint" type="fixed">
       <origin xyz="${x_loc} ${y_loc} ${z_loc}" rpy="0 0 0"/>
@@ -54,5 +54,5 @@
       </inertial>
     </link>
-  </xacro:macro>
+  </xacro:macro> -->
   <!--
     Stack macro - all the components relative transforms are made with respect
@@ -89,9 +89,9 @@
       </inertial>
     </link>
-    <xacro:stack_top_pole parent="${parent}" number="0" x_loc= "0.07" y_loc= "0.10" z_loc="0.210"/>
+    <!-- <xacro:stack_top_pole parent="${parent}" number="0" x_loc= "0.07" y_loc= "0.10" z_loc="0.210"/>
     <xacro:stack_top_pole parent="${parent}" number="1" x_loc= "0.07" y_loc= "-0.10" z_loc="0.210"/>
     <xacro:stack_top_pole parent="${parent}" number="2" x_loc= "-0.07" y_loc= "0.10" z_loc="0.210"/>
-    <xacro:stack_top_pole parent="${parent}" number="3" x_loc= "-0.07" y_loc= "-0.10" z_loc="0.210"/>
-    <joint name="plate_top_joint" type="fixed">
+    <xacro:stack_top_pole parent="${parent}" number="3" x_loc= "-0.07" y_loc= "-0.10" z_loc="0.210"/> -->
+    <!-- <joint name="plate_top_joint" type="fixed">
       <origin xyz="0 0 0.264" rpy="0 0 0"/>
       <parent link="${parent}"/>
@@ -116,5 +116,5 @@
         <inertia ixx="0.003328" ixy="0.0" ixz="0.0" iyy="0.003328" iyz="0.0" izz="0.006656" />
       </inertial>
-    </link>
+    </link> -->
   </xacro:macro>
 </robot>

File: lubobot/urdf/imu.urdf.xacro (robot description, xacro)
@@ -3,4 +3,7 @@
     xmlns:xacro="http://ros.org/wiki/xacro">
     <xacro:macro name="imu_sensor" params="xyz rpy parent">
+        <material name="red">
+            <color rgba="1 0 0 1"/>
+        </material>
         <joint name="imu_sensor_joint" type="fixed">
             <axis xyz="0 0 1" />
@@ -21,5 +24,5 @@
                     <box size="0.02 0.02 0.02"/>
                 </geometry>
-                <material name="iRobot/Red"/>
+                <material name="red"/>
             </visual>
             <inertial>

File: lubobot/urdf/lubobot.urdf.xacro (robot description, xacro)
@@ -2,14 +2,11 @@
 <robot xmlns:xacro="http://ros.org/wiki/xacro" name="lubobot_description">
 	<xacro:include filename="$(find lubobot)/urdf/body.urdf.xacro"/>
-	<xacro:include filename="$(find lubobot)/urdf/create_base.urdf.xacro" />
+	<xacro:include filename="$(find create_description)/urdf/create_2.urdf.xacro" />
 	<xacro:include filename="$(find lubobot)/urdf/imu.urdf.xacro" />
-	<xacro:include filename="$(find lubobot)/urdf/kinect.urdf.xacro"/>
-	<xacro:create_base wheel_separation="0.235" base_diameter="0.3485">
-		<mesh filename="package://lubobot/meshes/create_2.dae" />
-	</xacro:create_base>
+	<!-- <xacro:include filename="$(find lubobot)/urdf/kinect.urdf.xacro"/> -->
 	<xacro:body parent="base_link"/>
-	<xacro:kinect name="camera" parent="base_link">
+	<!-- <xacro:kinect name="camera" parent="base_link">
 		<origin xyz="0.050 0.033 0.210" rpy="0 0 0"/>
-	</xacro:kinect>
+	</xacro:kinect> -->
 	<xacro:imu_sensor xyz="0 0 0" rpy="0 0 0" parent="base_link" />
 </robot>
