Commit message: Added CAD models for URDF

File: lubobot/urdf/lubobot.urdf.xacro (robot description, xacro)
@@ -1,10 +1,14 @@
 <?xml version="1.0"?>
 <robot xmlns:xacro="http://ros.org/wiki/xacro" name="lubobot_description">
-	<xacro:include filename="$(find lubobot)/urdf/kinect.urdf.xacro"/>
+	<xacro:include filename="$(find lubobot)/urdf/body.urdf.xacro"/>
 	<xacro:include filename="$(find lubobot)/urdf/create_base.urdf.xacro" />
 	<xacro:include filename="$(find lubobot)/urdf/imu.urdf.xacro" />
+	<xacro:include filename="$(find lubobot)/urdf/kinect.urdf.xacro"/>
 	<xacro:create_base wheel_separation="0.235" base_diameter="0.3485">
 		<mesh filename="package://lubobot/meshes/create_2.dae" />
 	</xacro:create_base>
+	<xacro:body parent="base_link">
+		<origin xyz="0 0 0" rpy="0 0 0"/>
+	</xacro:body>
 	<xacro:kinect name="camera" parent="base_link">
 		<origin xyz="0 0 0.3" rpy="0 0 0"/>

Commit message: Replace kinect with LDS lidar

File: lubobot/urdf/lubobot.urdf.xacro (robot description, xacro)
@@ -4,9 +4,7 @@
 	<xacro:include filename="$(find create_description)/urdf/create_2.urdf.xacro" />
 	<xacro:include filename="$(find lubobot)/urdf/imu.urdf.xacro" />
-	<!-- <xacro:include filename="$(find lubobot)/urdf/kinect.urdf.xacro"/> -->
+	<xacro:include filename="$(find lubobot)/urdf/lds_lidar.urdf.xacro" />
 	<xacro:body parent="base_link"/>
-	<!-- <xacro:kinect name="camera" parent="base_link">
-		<origin xyz="0.050 0.033 0.210" rpy="0 0 0"/>
-	</xacro:kinect> -->
+	<xacro:lds_lidar xyz="0 0 0.19" rpy="0 0 ${3.1415}" parent="base_link" />
 	<xacro:imu_sensor xyz="0 0 0" rpy="0 0 0" parent="base_link" />
 </robot>
