Commit message: Remove unnecessary files; Update urdf.xacro

File: urdf/assembly_mount.urdf.xacro (robot description, xacro)
@@ -1,4 +1,4 @@
 <?xml version="1.0"?>
-<robot name="body"
+<robot name="assembly_mount"
   xmlns:xacro="http://ros.org/wiki/xacro">
   <!-- Heavily based on: https://github.com/turtlebot/turtlebot/blob/5a97fdd2661354a866ee41238e2197244c220840/turtlebot_description/urdf/stacks/hexagons.urdf.xacro -->
@@ -60,5 +60,5 @@
     other, but there is no necessary reason to do so.
   -->
-  <xacro:macro name="body" params="parent">
+  <xacro:macro name="assembly_mount" params="parent">
     <xacro:stack_bottom_pole parent="${parent}" number="0" x_loc= "0.08" y_loc= "0.08" z_loc="0.112"/>
     <xacro:stack_bottom_pole parent="${parent}" number="1" x_loc= "0.08" y_loc= "-0.08" z_loc="0.112"/>

File: urdf/lubobot.urdf.xacro (robot description, xacro)
@@ -1,10 +1,10 @@
 <?xml version="1.0"?>
 <robot xmlns:xacro="http://ros.org/wiki/xacro" name="lubobot_description">
-	<xacro:include filename="$(find lubobot)/urdf/body.urdf.xacro"/>
 	<xacro:include filename="$(find create_description)/urdf/create_2.urdf.xacro" />
+	<xacro:include filename="$(find lubobot)/urdf/assembly_mount.urdf.xacro"/>
 	<xacro:include filename="$(find lubobot)/urdf/imu.urdf.xacro" />
 	<xacro:include filename="$(find lubobot)/urdf/lds_lidar.urdf.xacro" />
-	<xacro:body parent="base_link"/>
+	<xacro:assembly_mount parent="base_link"/>
 	<xacro:lds_lidar xyz="0 0 0.19" rpy="0 0 ${3.1415}" parent="base_link" />
-	<xacro:imu_sensor xyz="0 0 0" rpy="0 0 0" parent="base_link" />
+	<xacro:imu_sensor xyz="0 -0.05 0" rpy="0 0 0" parent="base_link" />
 </robot>

Commit message: Body color is now grey

File: urdf/assembly_mount.urdf.xacro (robot description, xacro)
@@ -4,4 +4,7 @@
   <!-- Heavily based on: https://github.com/turtlebot/turtlebot/blob/5a97fdd2661354a866ee41238e2197244c220840/turtlebot_description/urdf/stacks/hexagons.urdf.xacro -->
   <xacro:macro name="stack_bottom_pole" params="parent number x_loc y_loc z_loc">
+    <material name="dark_gray">
+      <color rgba="0.2 0.2 0.2 1"/>
+    </material>
     <joint name="pole_bottom_${number}_joint" type="fixed">
       <origin xyz="${x_loc} ${y_loc} ${z_loc}" rpy="0 0 0"/>
@@ -15,4 +18,5 @@
           <mesh filename="package://lubobot/meshes/pole_80mm.stl" scale="0.001 0.001 0.001"/>
         </geometry>
+        <material name="dark_gray"/>
       </visual>
       <collision>
@@ -41,4 +45,5 @@
           <mesh filename="package://lubobot/meshes/pole_100mm.stl" scale="0.001 0.001 0.001"/>
         </geometry>
+        <material name="dark_gray"/>
       </visual>
       <collision>
@@ -76,4 +81,5 @@
           <mesh filename="package://lubobot/meshes/bottom_plate_290mm.stl" scale="0.001 0.001 0.001"/>
         </geometry>
+        <material name="dark_gray"/>
       </visual>
       <collision>
@@ -104,4 +110,5 @@
           <mesh filename="package://lubobot/meshes/top_plate_290mm.stl" scale="0.001 0.001 0.001"/>
         </geometry>
+        <material name="dark_gray"/>
       </visual>
       <collision>

Commit message: Renamed a few links to match convention

File: urdf/assembly_mount.urdf.xacro (robot description, xacro)
@@ -33,36 +33,4 @@
     </link>
   </xacro:macro>
-  <!-- <xacro:macro name="stack_top_pole" params="parent number x_loc y_loc z_loc">
-    <joint name="pole_top_${number}_joint" type="fixed">
-      <origin xyz="${x_loc} ${y_loc} ${z_loc}" rpy="0 0 0"/>
-      <parent link="${parent}"/>
-      <child link="pole_top_${number}_link"/>
-    </joint>
-    <link name="pole_top_${number}_link">
-      <visual>
-        <origin xyz=" 0 0 0" rpy="0 0 0"/>
-        <geometry>
-          <mesh filename="package://lubobot/meshes/pole_100mm.stl" scale="0.001 0.001 0.001"/>
-        </geometry>
-        <material name="dark_gray"/>
-      </visual>
-      <collision>
-        <origin xyz=" 0 0 0" rpy="0 0 0"/>
-        <geometry>
-          <mesh filename="package://lubobot/meshes/pole_100mm.stl" scale="0.001 0.001 0.001"/>
-        </geometry>
-      </collision>
-      <inertial>
-        <mass value="0.060"/>
-        <origin xyz="0 0 0"/>
-        <inertia ixx="0.000206991" ixy="0.0" ixz="0.0" iyy="0.000206991" iyz="0.0" izz="0.000001080"/>
-      </inertial>
-    </link>
-  </xacro:macro> -->
-  <!--
-    Stack macro - all the components relative transforms are made with respect
-    to the parent link (usually base_link). They could be made relative to each
-    other, but there is no necessary reason to do so.
-  -->
   <xacro:macro name="assembly_mount" params="parent">
     <xacro:stack_bottom_pole parent="${parent}" number="0" x_loc= "0.08" y_loc= "0.08" z_loc="0.112"/>
@@ -95,33 +63,4 @@
       </inertial>
     </link>
-    <!-- <xacro:stack_top_pole parent="${parent}" number="0" x_loc= "0.07" y_loc= "0.10" z_loc="0.210"/>
-    <xacro:stack_top_pole parent="${parent}" number="1" x_loc= "0.07" y_loc= "-0.10" z_loc="0.210"/>
-    <xacro:stack_top_pole parent="${parent}" number="2" x_loc= "-0.07" y_loc= "0.10" z_loc="0.210"/>
-    <xacro:stack_top_pole parent="${parent}" number="3" x_loc= "-0.07" y_loc= "-0.10" z_loc="0.210"/> -->
-    <!-- <joint name="plate_top_joint" type="fixed">
-      <origin xyz="0 0 0.264" rpy="0 0 0"/>
-      <parent link="${parent}"/>
-      <child link="plate_top_link"/>
-    </joint>
-    <link name="plate_top_link">
-      <visual>
-        <origin xyz="0 0 0" rpy="0 0 0"/>
-        <geometry>
-          <mesh filename="package://lubobot/meshes/top_plate_290mm.stl" scale="0.001 0.001 0.001"/>
-        </geometry>
-        <material name="dark_gray"/>
-      </visual>
-      <collision>
-        <origin xyz="0 0 0" rpy="0 0 0"/>
-        <geometry>
-          <mesh filename="package://lubobot/meshes/top_plate_290mm.stl" scale="0.001 0.001 0.001"/>
-        </geometry>
-      </collision>
-      <inertial>
-        <mass value="0.520"/>
-        <origin xyz="0 0 0"/>
-        <inertia ixx="0.003328" ixy="0.0" ixz="0.0" iyy="0.003328" iyz="0.0" izz="0.006656" />
-      </inertial>
-    </link> -->
   </xacro:macro>
 </robot>

File: urdf/imu.urdf.xacro (robot description, xacro)
@@ -6,11 +6,11 @@
             <color rgba="1 0 0 1"/>
         </material>
-        <joint name="imu_sensor_joint" type="fixed">
+        <joint name="imu_joint" type="fixed">
             <axis xyz="0 0 1" />
             <origin xyz="${xyz}" rpy="${rpy}"/>
             <parent link="${parent}"/>
-            <child link="imu_sensor_link"/>
+            <child link="imu_link"/>
         </joint>
-        <link name="imu_sensor_link">
+        <link name="imu_link">
             <collision>
                 <origin xyz="0 0 0" rpy="0 0 0"/>

File: urdf/lubobot.urdf.xacro (robot description, xacro)
@@ -3,8 +3,8 @@
 	<xacro:include filename="$(find create_description)/urdf/create_2.urdf.xacro" />
 	<xacro:include filename="$(find lubobot)/urdf/assembly_mount.urdf.xacro"/>
-	<xacro:include filename="$(find lubobot)/urdf/imu.urdf.xacro" />
-	<xacro:include filename="$(find lubobot)/urdf/lds_lidar.urdf.xacro" />
+	<!-- <xacro:include filename="$(find lubobot)/urdf/imu.urdf.xacro" />
+	<xacro:include filename="$(find lubobot)/urdf/lds_lidar.urdf.xacro" /> -->
 	<xacro:assembly_mount parent="base_link"/>
-	<xacro:lds_lidar xyz="0 0 0.19" rpy="0 0 ${3.1415}" parent="base_link" />
-	<xacro:imu_sensor xyz="0 -0.05 0" rpy="0 0 0" parent="base_link" />
+	<!-- <xacro:lds_lidar xyz="0 0 0.19" rpy="0 0 ${3.1415}" parent="base_link" />
+	<xacro:imu_sensor xyz="0 -0.05 0" rpy="0 0 0" parent="base_link" /> -->
 </robot>

Commit message: Implement basic gmapping

File: urdf/assembly_mount.urdf.xacro (robot description, xacro)
@@ -4,7 +4,4 @@
   <!-- Heavily based on: https://github.com/turtlebot/turtlebot/blob/5a97fdd2661354a866ee41238e2197244c220840/turtlebot_description/urdf/stacks/hexagons.urdf.xacro -->
   <xacro:macro name="stack_bottom_pole" params="parent number x_loc y_loc z_loc">
-    <material name="dark_gray">
-      <color rgba="0.2 0.2 0.2 1"/>
-    </material>
     <joint name="pole_bottom_${number}_joint" type="fixed">
       <origin xyz="${x_loc} ${y_loc} ${z_loc}" rpy="0 0 0"/>
@@ -18,5 +15,5 @@
           <mesh filename="package://lubobot/meshes/pole_80mm.stl" scale="0.001 0.001 0.001"/>
         </geometry>
-        <material name="dark_gray"/>
+        <material name="metal"/>
       </visual>
       <collision>
@@ -49,5 +46,5 @@
           <mesh filename="package://lubobot/meshes/bottom_plate_290mm.stl" scale="0.001 0.001 0.001"/>
         </geometry>
-        <material name="dark_gray"/>
+        <material name="wood"/>
       </visual>
       <collision>

File: urdf/lds_lidar.urdf.xacro (robot description, xacro)
@@ -3,7 +3,4 @@
     xmlns:xacro="http://ros.org/wiki/xacro">
     <xacro:macro name="lds_lidar" params="xyz rpy parent">
-      <material name="dark_gray">
-        <color rgba="0.2 0.2 0.2 1"/>
-      </material>
     <joint name="lidar_joint" type="fixed">
       <origin xyz="${xyz}" rpy="${rpy}"/>

File: urdf/lubobot.urdf.xacro (robot description, xacro)
@@ -1,10 +1,19 @@
 <?xml version="1.0"?>
 <robot xmlns:xacro="http://ros.org/wiki/xacro" name="lubobot_description">
+	<material name="dark_gray">
+      <color rgba="0.2 0.2 0.2 1"/>
+	</material>
+	<material name="wood">
+	  <color rgba="0.76 0.6 0.42 1"/>
+	</material>
+	<material name="metal">
+	  <color rgba="0.8 0.8 0.8 1"/>
+	</material>
 	<xacro:include filename="$(find create_description)/urdf/create_2.urdf.xacro" />
 	<xacro:include filename="$(find lubobot)/urdf/assembly_mount.urdf.xacro"/>
-	<!-- <xacro:include filename="$(find lubobot)/urdf/imu.urdf.xacro" />
-	<xacro:include filename="$(find lubobot)/urdf/lds_lidar.urdf.xacro" /> -->
+	<!-- <xacro:include filename="$(find lubobot)/urdf/imu.urdf.xacro" /> -->
+	<xacro:include filename="$(find lubobot)/urdf/lds_lidar.urdf.xacro" />
 	<xacro:assembly_mount parent="base_link"/>
-	<!-- <xacro:lds_lidar xyz="0 0 0.19" rpy="0 0 ${3.1415}" parent="base_link" />
-	<xacro:imu_sensor xyz="0 -0.05 0" rpy="0 0 0" parent="base_link" /> -->
+	<xacro:lds_lidar xyz="0 0 0.19" rpy="0 0 ${3.1415}" parent="base_link" />
+	<!-- <xacro:imu_sensor xyz="0 -0.05 0" rpy="0 0 0" parent="base_link" /> -->
 </robot>
