Commit message: Fix IMU pose configuration in urdf

File: urdf/imu.urdf.xacro (robot description, xacro)
@@ -16,5 +16,5 @@
                 <origin xyz="0 0 0" rpy="0 0 0"/>
                 <geometry>
-                    <box size="0.02 0.02 0.02"/>
+                    <box size="0.02 0.02 0.005"/>
                 </geometry>
             </collision>
@@ -22,5 +22,5 @@
                 <origin xyz="0 0 0" rpy="0 0 0"/>
                 <geometry>
-                    <box size="0.02 0.02 0.02"/>
+                    <box size="0.02 0.02 0.005"/>
                 </geometry>
                 <material name="red"/>

File: urdf/lubobot.urdf.xacro (robot description, xacro)
@@ -16,4 +16,4 @@
         <xacro:assembly_mount parent="base_link"/>
         <xacro:lds_lidar xyz="0 0 0.19" rpy="0 0 3.1415" parent="base_link"/>
-        <xacro:imu_sensor xyz="0 -0.1 0" rpy="0 0 0" parent="base_link" />
+        <xacro:imu_sensor xyz="0 0.105 0.074" rpy="0 0 0" parent="base_link" />
 </robot>
